Commit message: fix urdf

File: boden_description/urdf/model.urdf.xacro (robot description, xacro)
@@ -1,3 +1,4 @@
-<robot name="assem" version="1.0">
+<?xml version="1.0"?>
+<robot xmlns:xacro="http://ros.org/wiki/xacro">
   <joint name="Cube_link_joint" type="fixed">
     <origin rpy="0.00000 0.00000 0.00000" xyz="0.01837 -0.07980 -0.04656"/>
@@ -112,5 +113,5 @@
       <material name="Metal10"/>
       <geometry>
-        <mesh filename="package://meshes/dae/LongMotorAssem_V4 - Rough Shaft_V2-1.001.dae" scale="1.00000 1.00000 1.00000"/>
+          <mesh filename="file://$(find boden_description)/meshes/dae/LongMotorAssem_V4-RoughShaft_V2-1.001.dae" scale="1.00000 1.00000 1.00000"/>
       </geometry>
     </visual>
@@ -132,5 +133,5 @@
       <material name="Metal10"/>
       <geometry>
-        <mesh filename="package://meshes/dae/LongMotorAssem_V4 - Rough Shaft_V2-1.002.dae" scale="1.00000 1.00000 1.00000"/>
+          <mesh filename="file://$(find boden_description)/meshes/dae/LongMotorAssem_V4-RoughShaft_V2-1.002.dae" scale="1.00000 1.00000 1.00000"/>
       </geometry>
     </visual>
@@ -152,5 +153,5 @@
       <material name="Metal10"/>
       <geometry>
-        <mesh filename="package://meshes/dae/LongMotorAssem_V4 - Rough Shaft_V2-1.003.dae" scale="1.00000 1.00000 1.00000"/>
+        <mesh filename="file://$(find boden_description)/meshes/dae/LongMotorAssem_V4-RoughShaft_V2-1.003.dae" scale="1.00000 1.00000 1.00000"/>
       </geometry>
     </visual>
@@ -172,5 +173,5 @@
       <material name="Metal10"/>
       <geometry>
-        <mesh filename="package://meshes/dae/LongMotorAssem_V4 - Rough Shaft_V2-1.004.dae" scale="1.00000 1.00000 1.00000"/>
+        <mesh filename="file://$(find boden_description)/meshes/dae/LongMotorAssem_V4-RoughShaft_V2-1.004.dae" scale="1.00000 1.00000 1.00000"/>
       </geometry>
     </visual>
@@ -192,5 +193,5 @@
       <material name="Metal10"/>
       <geometry>
-        <mesh filename="package://meshes/dae/LongMotorAssem_V4 - Rough Shaft_V2-1.006.dae" scale="1.00000 1.00000 1.00000"/>
+        <mesh filename="file://$(find boden_description)/meshes/dae/LongMotorAssem_V4-RoughShaft_V2-1.006.dae" scale="1.00000 1.00000 1.00000"/>
       </geometry>
     </visual>
@@ -212,5 +213,5 @@
       <material name="Metal10"/>
       <geometry>
-        <mesh filename="package://meshes/dae/LongMotorAssem_V4 - Rough Shaft_V2-1.dae" scale="1.00000 1.00000 1.00000"/>
+        <mesh filename="file://$(find boden_description)/meshes/dae/LongMotorAssem_V4-RoughShaft_V2-1.dae" scale="1.00000 1.00000 1.00000"/>
       </geometry>
     </visual>
@@ -226,5 +227,5 @@
       <material name="Glass"/>
       <geometry>
-        <mesh filename="package://meshes/dae/Zed2-i.dae" scale="1.00000 1.00000 1.00000"/>
+        <mesh filename="file://$(find boden_description)/meshes/dae/Zed2-i.dae" scale="1.00000 1.00000 1.00000"/>
       </geometry>
     </visual>
@@ -240,5 +241,5 @@
       <material name="Metal28"/>
       <geometry>
-        <mesh filename="package://meshes/dae/chassisAssembly - chassisFrameShort-2.dae" scale="1.00000 1.00000 1.00000"/>
+        <mesh filename="file://$(find boden_description)/meshes/dae/chassisAssembly-chassisFrameShort-2.dae" scale="1.00000 1.00000 1.00000"/>
       </geometry>
     </visual>
@@ -254,5 +255,5 @@
       <material name="Plastic03"/>
       <geometry>
-        <mesh filename="package://meshes/dae/chassisAssembly - electronicsHousing-1 Rough 6 Pin Pannel C.001.dae" scale="1.00000 1.00000 1.00000"/>
+        <mesh filename="file://$(find boden_description)/meshes/dae/chassisAssembly-electronicsHousing-1-Rough-6-Pin-Pannel-C.001.dae" scale="1.00000 1.00000 1.00000"/>
       </geometry>
     </visual>
@@ -268,5 +269,5 @@
       <material name="Plastic04"/>
       <geometry>
-        <mesh filename="package://meshes/dae/chassisAssembly - roverBattery-1.dae" scale="1.00000 1.00000 1.00000"/>
+        <mesh filename="file://$(find boden_description)/meshes/dae/chassisAssembly-roverBattery-1.dae" scale="1.00000 1.00000 1.00000"/>
       </geometry>
     </visual>
@@ -282,5 +283,5 @@
       <material name="Plastic04"/>
       <geometry>
-        <mesh filename="package://meshes/dae/chassisAssembly - sensorPackageEnclosure-1.dae" scale="1.00000 1.00000 1.00000"/>
+        <mesh filename="file://$(find boden_description)/meshes/dae/chassisAssembly-sensorPackageEnclosure-1.dae" scale="1.00000 1.00000 1.00000"/>
       </geometry>
     </visual>
@@ -296,5 +297,5 @@
       <material name="Metal28"/>
       <geometry>
-        <mesh filename="package://meshes/dae/suspensionAssemblyMirror - RockerArmBack-7.001.dae" scale="1.00000 1.00000 1.00000"/>
+        <mesh filename="file://$(find boden_description)/meshes/dae/suspensionAssemblyMirror-RockerArmBack-7.001.dae" scale="1.00000 1.00000 1.00000"/>
       </geometry>
     </visual>
@@ -310,5 +311,5 @@
       <material name="Metal28"/>
       <geometry>
-        <mesh filename="package://meshes/dae/suspensionAssemblyMirror - RockerArmBack-7.dae" scale="1.00000 1.00000 1.00000"/>
+        <mesh filename="file://$(find boden_description)/meshes/dae/suspensionAssemblyMirror-RockerArmBack-7.dae" scale="1.00000 1.00000 1.00000"/>
       </geometry>
     </visual>
@@ -324,5 +325,5 @@
       <material name="Metal28"/>
       <geometry>
-        <mesh filename="package://meshes/dae/suspensionAssemblyMirror - bogieCenterBracket_Outside-6.001.dae" scale="1.00000 1.00000 1.00000"/>
+        <mesh filename="file://$(find boden_description)/meshes/dae/suspensionAssemblyMirror-bogieCenterBracket_Outside-6.001.dae" scale="1.00000 1.00000 1.00000"/>
       </geometry>
     </visual>
@@ -338,5 +339,5 @@
       <material name="Metal28"/>
       <geometry>
-        <mesh filename="package://meshes/dae/suspensionAssemblyMirror - bogieCenterBracket_Outside-6.dae" scale="1.00000 1.00000 1.00000"/>
+        <mesh filename="file://$(find boden_description)/meshes/dae/suspensionAssemblyMirror-bogieCenterBracket_Outside-6.dae" scale="1.00000 1.00000 1.00000"/>
       </geometry>
     </visual>
