Commit message: tune new webots simulation

File: boden_description/urdf/boden_description.urdf (robot description, URDF)
Before this commit: robot boden_description, 16 links, 15 joints
Links:
- link Zed2i_link: geometry visual mesh filename=package://boden_description/meshes/dae/Zed2i.dae scale=1.00000 1.00000 1.00000
- link battery_link: geometry visual mesh filename=package://boden_description/meshes/dae/battery.dae scale=1.00000 1.00000 1.00000
- link electronics_link: geometry visual mesh filename=package://boden_description/meshes/dae/electronics.dae scale=1.00000 1.00000 1.00000
- link left_wheel_1_link: geometry collision cylinder length=0.10744 radius=0.13329; visual mesh filename=package://boden_description/meshes/dae/wheel-left.dae scale=1.00000 1.00000 1.00000
- link left_wheel_2_link: geometry collision cylinder length=0.10744 radius=0.13329; visual mesh filename=package://boden_description/meshes/dae/wheel-left.dae scale=1.00000 1.00000 1.00000
- link left_wheel_3_link: geometry collision cylinder length=0.10744 radius=0.13329; visual mesh filename=package://boden_description/meshes/dae/wheel-left.dae scale=1.00000 1.00000 1.00000
- link main_plate_link: geometry visual mesh filename=package://boden_description/meshes/dae/main-plate.dae scale=1.00000 1.00000 1.00000
- link right_wheel_1_link: geometry collision cylinder length=0.10744 radius=0.13329; visual mesh filename=package://boden_description/meshes/dae/wheel-right.dae scale=1.00000 1.00000 1.00000
- link right_wheel_2_link: geometry collision cylinder length=0.10744 radius=0.13329; visual mesh filename=package://boden_description/meshes/dae/wheel-right.dae scale=1.00000 1.00000 1.00000
- link right_wheel_3_link: geometry collision cylinder length=0.10744 radius=0.13335; visual mesh filename=package://boden_description/meshes/dae/wheel-right.dae scale=1.00000 1.00000 1.00000
- link sensor_package_link: geometry visual mesh filename=package://boden_description/meshes/dae/sensor-package.dae scale=1.00000 1.00000 1.00000
- link suspension_left_main_link: geometry visual mesh filename=package://boden_description/meshes/dae/suspension-left.dae scale=1.00000 1.00000 1.00000
- link suspension_left_sub_link: geometry visual mesh filename=package://boden_description/meshes/dae/suspension-left-sub.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 scale=1.00000 1.00000 1.00000
- link suspension_right_main_link: geometry visual mesh filename=package://boden_description/meshes/dae/suspension-right.dae scale=1.00000 1.00000 1.00000
- link suspension_right_sub_link: geometry visual mesh filename=package://boden_description/meshes/dae/suspension-right-sub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 scale=1.00000 1.00000 1.00000

File: boden_description/urdf/boden_description_relpath.urdf (robot description, URDF)
Before this commit: robot boden_description, 16 links, 15 joints
Links:
- link Zed2i_link: geometry visual mesh filename=../boden_description/meshes/dae/Zed2i.dae scale=1.00000 1.00000 1.00000
- link battery_link: geometry visual mesh filename=../boden_description/meshes/dae/battery.dae scale=1.00000 1.00000 1.00000
- link electronics_link: geometry visual mesh filename=../boden_description/meshes/dae/electronics.dae scale=1.00000 1.00000 1.00000
- link left_wheel_1_link: geometry collision cylinder length=0.10744 radius=0.13329; visual mesh filename=../boden_description/meshes/dae/wheel-left.dae scale=1.00000 1.00000 1.00000
- link left_wheel_2_link: geometry collision cylinder length=0.10744 radius=0.13329; visual mesh filename=../boden_description/meshes/dae/wheel-left.dae scale=1.00000 1.00000 1.00000
- link left_wheel_3_link: geometry collision cylinder length=0.10744 radius=0.13329; visual mesh filename=../boden_description/meshes/dae/wheel-left.dae scale=1.00000 1.00000 1.00000
- link main_plate_link: geometry visual mesh filename=../boden_description/meshes/dae/main-plate.dae scale=1.00000 1.00000 1.00000
- link right_wheel_1_link: geometry collision cylinder length=0.10744 radius=0.13329; visual mesh filename=../boden_description/meshes/dae/wheel-right.dae scale=1.00000 1.00000 1.00000
- link right_wheel_2_link: geometry collision cylinder length=0.10744 radius=0.13329; visual mesh filename=../boden_description/meshes/dae/wheel-right.dae scale=1.00000 1.00000 1.00000
- link right_wheel_3_link: geometry collision cylinder length=0.10744 radius=0.13335; visual mesh filename=../boden_description/meshes/dae/wheel-right.dae scale=1.00000 1.00000 1.00000
- link sensor_package_link: geometry visual mesh filename=../boden_description/meshes/dae/sensor-package.dae scale=1.00000 1.00000 1.00000
- link suspension_left_main_link: geometry visual mesh filename=../boden_description/meshes/dae/suspension-left.dae scale=1.00000 1.00000 1.00000
- link suspension_left_sub_link: geometry visual mesh filename=../boden_description/meshes/dae/suspension-left-sub.dae scale=1.00000 1.00000 1.00000
- link suspension_right_main_link: geometry visual mesh filename=../boden_description/meshes/dae/suspension-right.dae scale=1.00000 1.00000 1.00000
- link suspension_right_sub_link: geometry visual mesh filename=../boden_description/meshes/dae/suspension-right-sub.dae scale=1.00000 1.00000 1.00000
