Commit message: configure ros2 control

File: bodenbot/description/ros2_control/bodenbot.ros2_control.xacro (robot description, xacro)
@@ -12,31 +12,27 @@
       <joint name="right_wheel_1_link_joint">
         <command_interface name="velocity"/>
-        <state_interface name="velocity">
-          <param name="initial_value">0.0</param>
-        </state_interface>
+        <state_interface name="velocity" />
+        <state_interface name="position" />
         <param name="id">0</param>
-        <param name="reversed">false</param>
+        <param name="reversed">true</param>
       </joint>
       <joint name="right_wheel_2_link_joint">
         <command_interface name="velocity"/>
-        <state_interface name="velocity">
-          <param name="initial_value">0.0</param>
-        </state_interface>
+        <state_interface name="velocity" />
+        <state_interface name="position" />
         <param name="id">1</param>
-        <param name="reversed">false</param>
+        <param name="reversed">true</param>
       </joint>
       <joint name="right_wheel_3_link_joint">
         <command_interface name="velocity"/>
-        <state_interface name="velocity">
-          <param name="initial_value">0.0</param>
-        </state_interface>
+        <state_interface name="velocity" />
+        <state_interface name="position" />
         <param name="id">2</param>
-        <param name="reversed">false</param>
+        <param name="reversed">true</param>
       </joint>
       <joint name="left_wheel_1_link_joint">
         <command_interface name="velocity"/>
-        <state_interface name="velocity">
-          <param name="initial_value">0.0</param>
-        </state_interface>
+        <state_interface name="velocity" />
+        <state_interface name="position" />
         <param name="id">3</param>
         <param name="reversed">false</param>
@@ -44,7 +40,6 @@
       <joint name="left_wheel_2_link_joint">
         <command_interface name="velocity"/>
-        <state_interface name="velocity">
-          <param name="initial_value">0.0</param>
-        </state_interface>
+        <state_interface name="velocity" />
+        <state_interface name="position" />
         <param name="id">4</param>
         <param name="reversed">false</param>
@@ -52,7 +47,6 @@
       <joint name="left_wheel_3_link_joint">
         <command_interface name="velocity"/>
-        <state_interface name="velocity">
-          <param name="initial_value">0.0</param>
-        </state_interface>
+        <state_interface name="velocity" />
+        <state_interface name="position" />
         <param name="id">5</param>
         <param name="reversed">false</param>

File: bodenbot/description/urdf/bodenbot_description.urdf.xacro (robot description, xacro)
@@ -3,5 +3,5 @@
 <xacro:macro name="bodenbot" params="prefix">
   <joint name="Zed2i_link_joint" type="fixed">
-    <origin rpy="1.57080 0.00000 -1.57080" xyz="-0.08420 0.00894 0.08299"/>
+    <origin rpy="0.00000 0.00682 3.14159" xyz="-0.08420 0.00894 0.08299"/>
     <parent link="electronics_link"/>
     <child link="Zed2i_link"/>
@@ -13,10 +13,10 @@
   </joint>
   <joint name="battery_link_joint" type="fixed">
-    <origin rpy="0.00000 0.00000 0.00000" xyz="0.05208 0.00000 0.05627"/>
+    <origin rpy="0.00000 0.00000 -3.14159" xyz="-0.09286 -0.00214 0.05627"/>
     <parent link="main_plate_link"/>
     <child link="battery_link"/>
   </joint>
   <joint name="electronics_link_joint" type="fixed">
-    <origin rpy="0.00000 0.00000 0.00000" xyz="-0.08592 -0.00513 0.10698"/>
+    <origin rpy="0.00000 0.00000 -3.14159" xyz="0.04514 0.00299 0.10698"/>
     <parent link="main_plate_link"/>
     <child link="electronics_link"/>
@@ -65,5 +65,5 @@
   </joint>
   <joint name="sensor_package_link_joint" type="fixed">
-    <origin rpy="-3.14159 0.00000 0.00000" xyz="-0.07970 -0.00236 -0.02071"/>
+    <origin rpy="-3.14159 0.00000 -3.14159" xyz="0.03892 0.00022 -0.02071"/>
     <parent link="main_plate_link"/>
     <child link="sensor_package_link"/>
@@ -72,5 +72,5 @@
     <limit lower="-0.50000" upper="0.50000" effort="1.50000" velocity="0.01500"/>
     <mimic multiplier="-1.00000" offset="0.00000" joint="suspension_right_main_link_joint"/>
-    <origin rpy="1.57080 0.00000 0.00000" xyz="0.00500 -0.16509 0.09549"/>
+    <origin rpy="1.57080 0.00000 -3.14159" xyz="-0.04578 0.16295 0.09549"/>
     <parent link="main_plate_link"/>
     <child link="suspension_left_main_link"/>
@@ -86,5 +86,5 @@
   <joint name="suspension_right_main_link_joint" type="revolute">
     <limit lower="-0.50000" upper="0.50000" effort="1.50000" velocity="0.01500"/>
-    <origin rpy="1.57080 -0.00000 3.14159" xyz="0.00509 0.16510 0.09582"/>
+    <origin rpy="1.57080 -0.00000 -0.00000" xyz="-0.04587 -0.16724 0.09582"/>
     <parent link="main_plate_link"/>
     <child link="suspension_right_main_link"/>
@@ -99,18 +99,4 @@
   </joint>
   <link name="Zed2i_link">
-    <sensor name="zed2i_camera" type="camera">
-      <origin rpy="0.00000 -0.00000 -0.00000" xyz="0.00000 0.00000 0.00000"/>
-      <parent link="Zed2i_link"/>
-      <camera>
-        <image>
-          <width>662</width>
-          <height>376</height>
-          <hfov>1.57080</hfov>
-        </image>
-      </camera>
-    </sensor>
-    <sensor name="gps" type="GPS">
-      <parent link="Zed2i_link"/>
-    </sensor>
     <inertial>
       <inertia ixx="0.00048" ixy="0.00000" ixz="0.00000" iyy="0.00004" iyz="0.00000" izz="0.00050"/>
@@ -119,5 +105,5 @@
     </inertial>
     <visual name="Zed2i_visual">
-      <origin rpy="3.14159 1.57079 3.14159" xyz="0.00000 0.00000 0.00000"/>
+      <origin rpy="1.57080 -0.00000 3.14159" xyz="-0.00000 -0.00000 -0.00000"/>
       <material name="Glass"/>
       <geometry>
@@ -154,5 +140,5 @@
     </inertial>
     <visual name="electronics_visual">
-      <origin rpy="1.57080 0.00000 0.00000" xyz="0.00000 0.00000 0.00000"/>
+      <origin rpy="1.57080 0.00000 0.00000" xyz="-0.00000 0.00000 0.00000"/>
       <material name="Plastic"/>
       <geometry>
@@ -163,16 +149,16 @@
   <link name="left_wheel_1_link">
     <collision name="left_wheel_1_collision">
+      <origin rpy="-0.00000 0.00000 0.00000" xyz="-0.00006 -0.00002 0.06622"/>
+      <geometry>
+        <cylinder radius="0.13329" length="0.10744"/>
+      </geometry>
+    </collision>
+    <inertial>
+      <inertia ixx="0.00162" ixy="0.00000" ixz="0.00000" iyy="0.00267" iyz="0.00000" izz="0.00162"/>
       <origin rpy="0.00000 0.00000 0.00000" xyz="-0.00006 -0.00002 0.06622"/>
-      <geometry>
-        <cylinder radius="0.13329" length="0.10744"/>
-      </geometry>
-    </collision>
-    <inertial>
-      <inertia ixx="0.00162" ixy="0.00000" ixz="0.00000" iyy="0.00267" iyz="0.00000" izz="0.00162"/>
-      <origin rpy="0.00000 0.00000 0.00000" xyz="-0.00006 -0.00002 0.06622"/>
       <mass value="0.30000"/>
     </inertial>
     <visual name="left_wheel_1_visual">
-      <origin rpy="0.00000 0.00000 0.00000" xyz="0.00000 -0.00000 -0.00000"/>
+      <origin rpy="-0.00000 0.00000 0.00000" xyz="-0.00000 0.00000 0.00000"/>
       <material name="Metal"/>
       <geometry>
@@ -224,9 +210,9 @@
     <inertial>
       <inertia ixx="0.00100" ixy="0.00000" ixz="0.00000" iyy="0.00100" iyz="0.00000" izz="0.00100"/>
-      <origin rpy="0.00000 0.00000 0.00000" xyz="-0.03928 0.00000 -0.00904"/>
+      <origin rpy="0.00000 0.00000 0.00000" xyz="-0.00150 -0.00214 -0.00904"/>
       <mass value="2.00000"/>
     </inertial>
     <visual name="main_plate_visual">
-      <origin rpy="1.57080 0.00000 0.00000" xyz="0.00000 0.00000 0.00674"/>
+      <origin rpy="1.57080 0.00000 -3.14159" xyz="-0.04078 -0.00214 0.00674"/>
       <material name="Metal"/>
       <geometry>
@@ -248,5 +234,5 @@
     </inertial>
     <visual name="right_wheel_1_visual">
-      <origin rpy="-3.14159 -0.00000 0.00000" xyz="0.00000 0.00000 0.00000"/>
+      <origin rpy="-3.14159 -0.00000 0.00000" xyz="-0.00000 -0.00000 -0.00000"/>
       <material name="Rubber"/>
       <geometry>
@@ -268,5 +254,5 @@
     </inertial>
     <visual name="right_wheel_2_visual">
-      <origin rpy="3.14159 0.00000 0.00000" xyz="-0.00000 -0.00000 0.00000"/>
+      <origin rpy="3.14159 0.00000 0.00000" xyz="0.00000 0.00000 -0.00000"/>
       <material name="Rubber"/>
       <geometry>
@@ -277,5 +263,5 @@
   <link name="right_wheel_3_link">
     <collision name="right_wheel_3_collision">
-      <origin rpy="-3.14159 -0.00000 0.00000" xyz="0.00001 0.00000 0.06622"/>
+      <origin rpy="-3.14159 -0.00000 0.00000" xyz="0.00001 -0.00000 0.06622"/>
       <geometry>
         <cylinder radius="0.13335" length="0.10744"/>
@@ -284,5 +270,5 @@
     <inertial>
       <inertia ixx="0.00162" ixy="0.00000" ixz="0.00000" iyy="0.00267" iyz="0.00000" izz="0.00162"/>
-      <origin rpy="0.00000 0.00000 0.00000" xyz="0.00001 0.00000 0.06622"/>
+      <origin rpy="0.00000 0.00000 0.00000" xyz="0.00001 -0.00000 0.06622"/>
       <mass value="0.30000"/>
     </inertial>
@@ -316,5 +302,5 @@
     </inertial>
     <visual name="suspension_left_main_visual">
-      <origin rpy="3.14159 0.00000 0.00000" xyz="0.00000 0.00000 -0.00000"/>
+      <origin rpy="3.14159 0.00000 0.00000" xyz="0.00000 0.00000 0.00000"/>
       <material name="Rubber"/>
       <geometry>
@@ -330,5 +316,5 @@
     </inertial>
     <visual name="suspension_left_sub_visual">
-      <origin rpy="3.14159 -0.00000 -0.00000" xyz="0.00000 0.00000 0.00000"/>
+      <origin rpy="3.14159 0.00000 -0.00000" xyz="-0.00000 -0.00000 0.00000"/>
       <material name="Rubber"/>
       <geometry>
@@ -358,5 +344,5 @@
     </inertial>
     <visual name="suspension_right_sub_visual">
-      <origin rpy="-0.00000 0.00000 0.00000" xyz="-0.00000 -0.00000 0.00000"/>
+      <origin rpy="-0.00000 0.00000 0.00000" xyz="0.00000 0.00000 -0.00000"/>
       <material name="Metal"/>
       <geometry>

Commit message: get i2c working

File: bodenbot/description/ros2_control/bodenbot.ros2_control.xacro (robot description, xacro)
@@ -15,5 +15,5 @@
         <state_interface name="position" />
         <param name="id">2</param>
-        <param name="reversed">true</param>
+        <param name="reversed">false</param>
       </joint>
       <joint name="right_wheel_2_link_joint">
@@ -22,5 +22,5 @@
         <state_interface name="position" />
         <param name="id">0</param>
-        <param name="reversed">true</param>
+        <param name="reversed">false</param>
       </joint>
       <joint name="right_wheel_3_link_joint">
@@ -29,5 +29,5 @@
         <state_interface name="position" />
         <param name="id">3</param>
-        <param name="reversed">true</param>
+        <param name="reversed">false</param>
       </joint>
       <joint name="left_wheel_1_link_joint">

File: bodenbot/description/urdf/bodenbot_description.urdf.xacro (robot description, xacro)
@@ -48,5 +48,5 @@
     <parent link="suspension_right_sub_link"/>
     <child link="right_wheel_1_link"/>
-    <axis xyz="0.00000 0.00000 1.00000"/>
+    <axis xyz="0.00000 0.00000 -1.00000"/>
   </joint>
   <joint name="right_wheel_2_link_joint" type="continuous">
@@ -55,5 +55,5 @@
     <parent link="suspension_right_sub_link"/>
     <child link="right_wheel_2_link"/>
-    <axis xyz="0.00000 0.00000 1.00000"/>
+    <axis xyz="0.00000 0.00000 -1.00000"/>
   </joint>
   <joint name="right_wheel_3_link_joint" type="continuous">
@@ -62,5 +62,5 @@
     <parent link="suspension_right_main_link"/>
     <child link="right_wheel_3_link"/>
-    <axis xyz="0.00000 0.00000 1.00000"/>
+    <axis xyz="0.00000 0.00000 -1.00000"/>
   </joint>
   <joint name="sensor_package_link_joint" type="fixed">
